File: smart-system-monitor-IoT_AI/smart-system-monitor-IoT_AI.kicad_sch (KiCad schematic)
At the start: 4 parts, among them U1 ESP32-WROOM-32, U2 INA219AxD, U3 TMP36xS

Commit message: Assembling
Parts:
- added BT1: 18650 2500-3500 mAh, symbol Device:Battery_Cell
- added C1: 0.1uF, symbol Device:C
- added U4: ~, symbol tp4056:TP4056
Connections:
- net GND: now also C1.2
- net at U3.1 (V_{OUT}): now also U1.6 (IO34)
- net at U3.4 (GND): now also C1.1
- new net: BT1.1 (+), U4.4 (B+)
- new net: BT1.2 (-), U4.5 (B-)
Other:
- moved on the sheet: U3
