File: smart-system-monitor-IoT_AI.kicad_sch (KiCad schematic)
At the start: 7 parts, among them U1 ESP32-WROOM-32, U2 INA219AxD, U3 TMP36xS

Commit message: Finishing up with schematics
Parts:
- removed DS1: OLED-128O064D, Display:OLED-128O064D, symbol Display_Graphic:OLED-128O064D
- added DS1: OLED_128X64, OLED_128X64_1.3_I2C:LCD_OLED_128X64_1.3_I2C, symbol OLED_128X64_1.3_I2C:OLED_128X64_1.3_I2C
Connections:
- net GND: now also U4.6 (OUT-), DS1.2 (GND)
- net at U3.8 (+Vs): now also U1.2 (VDD), U2.5 (VS), U4.3 (OUT+), DS1.1 (VDD)
- net at U1.33 (IO21), U2.3 (SDA): now also DS1.4 (SDA)
- net at U1.36 (IO22), U2.4 (SCL): now also DS1.3 (SCK)
- no-connect marks 0 -> 33
Other:
- company: (none) -> Vladyslav Hirchuk - git: SoloScriptSage
- title: (none) -> Smart System Monitor IoT with AI
- moved on the sheet: BT1, C1, U1, U2, U3, U4
